File: hardware/carrier/carrier.kicad_pcb (KiCad board)
At the start: 2 copper layers, 0 parts

Commit message: hardware: carrier rev A PCB first pass (placed, autorouted, DRC clean)
- carrier.kicad_pcb: 69.0 x 49.9 mm outline with R2 corners, module hole
  grid, 25 x 12 mm antenna keep-out on both layers; all parts on the
  outer face; footprints linked to schematic symbols (parity clean).
- Net classes in the project: Power 0.6 mm, GND 0.4 mm, signals 0.25 mm.
- GND: pours both layers, fan-out via per SMD GND pad, stitching vias;
  F.Cu track keep-outs under the J1/J3/J5 bodies.
- Signals autorouted with Freerouting 2.5 (DSN/SES), GND left to pours.
- Schematic: H1 (under the antenna) is now a bare NPTH; holes, solder
  jumpers and test points are excluded from the BOM.

DRC: 0 errors, 0 unconnected; only J1's library silk crossing the edge.

Co-Authored-By: Claude Opus 5.5 <noreply@anthropic.com>
Claude-Session: https://claude.ai/code/session_01JQabpaYYgc1UrT8JpxmMza
Parts:
- added C1: 5F 2.7V, Capacitor_THT:CP_Radial_D8.0mm_P3.50mm, F.Cu at (160.0, 113.0)
- added C2: 10u 16V, Capacitor_SMD:C_0805_2012Metric, F.Cu at (110.8, 126.0)
- added C3: 100n, Capacitor_SMD:C_0805_2012Metric, F.Cu at (112.4, 145.2)
- added C4: 5F 2.7V, Capacitor_THT:CP_Radial_D8.0mm_P3.50mm, F.Cu at (151.0, 113.0)
- added D1: SS34, Diode_SMD:D_SMA, F.Cu at (115.0, 131.0)
- added D2: SS34, Diode_SMD:D_SMA, F.Cu at (145.0, 131.5)
- added F1: PTC 1.1A hold, Fuse:Fuse_1812_4532Metric, F.Cu at (124.0, 140.6)
- added H1: M2.5 NPTH, MountingHole:MountingHole_2.7mm_M2.5, F.Cu at (104.5, 104.4)
- added H2: M2.5, MountingHole:MountingHole_2.7mm_M2.5_Pad, F.Cu at (164.5, 104.4)
- added H3: M2.5, MountingHole:MountingHole_2.7mm_M2.5_Pad, F.Cu at (104.5, 145.4)
- added H4: M2.5, MountingHole:MountingHole_2.7mm_M2.5_Pad, F.Cu at (164.5, 145.4)
- added J1: USB-C power only, Connector_USB:USB_C_Receptacle_HRO_TYPE-C-31-M-12, F.Cu at (132.0, 146.2)
- added J2: to PN532 (I2C), Connector_JST:JST_PH_S5B-PH-K_1x05_P2.00mm_Horizontal, F.Cu at (140.0, 107.4)
- added J3: to module J8, Connector_JST:JST_SH_SM12B-SRSS-TB_1x12-1MP_P1.00mm_Horizontal, F.Cu at (103.1, 131.0)
- added J4: UART debug, Connector_PinHeader_2.54mm:PinHeader_1x03_P2.54mm_Vertical, F.Cu at (162.0, 133.6)
- added J5: to module J1 (BAT), Connector_Molex:Molex_PicoBlade_53261-0271_1x02-1MP_P1.25mm_Horizontal, F.Cu at (166.2, 127.5)
- added JP1: bypass D1 (closed), Jumper:SolderJumper-2_P1.3mm_Bridged_RoundedPad1.0x1.5mm, F.Cu at (115.0, 134.6)
- added JP2: BAT->VCAP (closed), Jumper:SolderJumper-2_P1.3mm_Bridged_RoundedPad1.0x1.5mm, F.Cu at (160.6, 127.5)
- added R1: 100k 1%, Resistor_SMD:R_0805_2012Metric, F.Cu at (116.6, 140.4)
- added R2: 11k3 1%, Resistor_SMD:R_0805_2012Metric, F.Cu at (116.6, 144.2)
- added R3: 22R 1W, Resistor_SMD:R_2512_6332Metric, F.Cu at (145.0, 127.0)
- added R4: 10k, Resistor_SMD:R_0805_2012Metric, F.Cu at (158.2, 120.0)
- added R5: 10k, Resistor_SMD:R_0805_2012Metric, F.Cu at (149.2, 120.0)
- added R6: 5k1, Resistor_SMD:R_0805_2012Metric, F.Cu at (128.4, 137.6)
- added R7: 5k1, Resistor_SMD:R_0805_2012Metric, F.Cu at (135.6, 137.6)
- added R8: 4k7, Resistor_SMD:R_0805_2012Metric, F.Cu at (126.0, 133.5)
- added TP1: USB_5V, TestPoint:TestPoint_Pad_D1.5mm, F.Cu at (114.0, 126.0)
- added TP2: VCAP, TestPoint:TestPoint_Pad_D1.5mm, F.Cu at (163.0, 120.6)
- added TVS1: SMAJ5.0A, Diode_SMD:D_SMA, F.Cu at (120.5, 134.6)
- added U2: TPS3808G01DBV, Package_TO_SOT_SMD:SOT-23-6, F.Cu at (112.4, 141.6)
Routing:
- net +3V3: track 0.00 -> 69.5 mm, vias 0 -> 2
- net /UART_RX: track 0.00 -> 61.1 mm
- net /UART_TX: track 0.00 -> 57.4 mm, vias 0 -> 1
- net /USB_5V: track 0.00 -> 52.0 mm
- net /NFC_IRQ: track 0.00 -> 43.0 mm, vias 0 -> 2
- net /SDA: track 0.00 -> 42.1 mm, vias 0 -> 1
- net /SCL: track 0.00 -> 40.0 mm, vias 0 -> 1
- net /VCAP: track 0.00 -> 35.3 mm
- net GND: track 0.00 -> 28.6 mm, vias 0 -> 26
- net /VIN_CAR: track 0.00 -> 25.7 mm, vias 0 -> 2
- net /VIN_FUSED: track 0.00 -> 24.0 mm
- net /VCAP_MID: track 0.00 -> 20.2 mm
- net /PWR_SENSE: track 0.00 -> 7.88 mm
- net /SENSE_DIV: track 0.00 -> 4.99 mm
- net /USB_CC1: track 0.00 -> 4.78 mm
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- added copper zone on B.Cu, net GND
- added copper zone on F.Cu, net GND
Other:
- board outline added: 69 x 49.9 mm
- board text added: "2x 5F 2.7V supercaps"
- board text added: "ANTENNA"
- board text added: "JP1 bridged = D1 bypassed"
- board text added: "JP2 bridged = BAT->caps"
- board text added: "KEEP-OUT"
- board text added: "car-km carrier rev A"
