File: hardware/carrier/carrier.kicad_sch (KiCad schematic)
At the start: 30 parts, among them J1 USB-C power only, J2 to PN532 (I2C), J3 to module J8, J4 UART debug, J5 to module J1 (BAT), U2 TPS3808G01DBV

Commit message: hardware: carrier rev A PCB first pass (placed, autorouted, DRC clean)
- carrier.kicad_pcb: 69.0 x 49.9 mm outline with R2 corners, module hole
  grid, 25 x 12 mm antenna keep-out on both layers; all parts on the
  outer face; footprints linked to schematic symbols (parity clean).
- Net classes in the project: Power 0.6 mm, GND 0.4 mm, signals 0.25 mm.
- GND: pours both layers, fan-out via per SMD GND pad, stitching vias;
  F.Cu track keep-outs under the J1/J3/J5 bodies.
- Signals autorouted with Freerouting 2.5 (DSN/SES), GND left to pours.
- Schematic: H1 (under the antenna) is now a bare NPTH; holes, solder
  jumpers and test points are excluded from the BOM.

DRC: 0 errors, 0 unconnected; only J1's library silk crossing the edge.

Co-Authored-By: Claude Opus 5.5 <noreply@anthropic.com>
Claude-Session: https://claude.ai/code/session_01JQabpaYYgc1UrT8JpxmMza
Parts:
- removed H1: M2.5, MountingHole:MountingHole_2.7mm_M2.5_Pad, symbol Mechanical:MountingHole_Pad
- added H1: M2.5 NPTH, MountingHole:MountingHole_2.7mm_M2.5, symbol Mechanical:MountingHole
- H2, H3, H4, JP1, JP2, TP1, TP2: now left out of the parts list
Other:
- note added: "H1 = top-left hole, inside the antenna keep-out"
